File: ez-bno055.kicad_pcb (KiCad board)
At the start: 2 copper layers, 20.4 x 30 mm, 29 parts, among them J1 Conn_01x06, J2 Conn_01x06, J3 I2C, J4 I2C, U1 BNO055, U2 AP2112K-3.3, Y1 32.768KHz

Commit message: Changes crystal to 3215 size
Parts:
- Y1: footprint Crystal:Crystal_SMD_5032-2Pin_5.0x3.2mm -> Crystal:Crystal_SMD_3215-2Pin_3.2x1.5mm
- moved C8 3.10 mm to (138.3, 94.1), turned to 180 degrees
- moved C7 3.08 mm to (140.3, 94.1), turned to 0 degrees
- moved Y1 0.56 mm to (139.3, 92.4), turned to 180 degrees
Routing:
- net Net-(U1-XIN32): track 5.30 -> 3.81 mm
- net Net-(U1-XOUT32): track 5.26 -> 3.81 mm
Other:
- board text added: "3V3"
- board text added: "ADR"
- board text added: "GND"
- board text added: "I2C_ADDR"
- board text added: "I2C_RPU"
- board text added: "INT"
- board text added: "PS0"
- board text added: "PS1"
- board text added: "SCL"
- board text added: "SDA"
- board text added: "VIN"
- board text added: "X"
- board text added: "Y"
- board text added: "Z"
- board text added: "~{RST}"
