File: ez-bno055.kicad_sch (KiCad schematic)
At the start: 29 parts, among them J1 Conn_01x06, J2 Conn_01x06, J3 I2C, J4 I2C, U1 BNO055, U2 AP2112K-3.3, Y1 32.768KHz

Commit message: Changes crystal to 3215 size
Parts:
- Y1: footprint Crystal:Crystal_SMD_5032-2Pin_5.0x3.2mm -> Crystal:Crystal_SMD_3215-2Pin_3.2x1.5mm
Changed lines of the file:
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@@
       (effects (font (size 1.27 1.27)) hide)
     )
-    (pin "2")
-    (pin "1")
+    (pin "1")
+    (pin "2")
     (instances
       (project "ez-bno055"
@@
       (effects (font (size 1.27 1.27)) (justify right))
     )
-    (property "Footprint" "Crystal:Crystal_SMD_5032-2Pin_5.0x3.2mm" (at 175.26 88.9 0)
+    (property "Footprint" "Crystal:Crystal_SMD_3215-2Pin_3.2x1.5mm" (at 175.26 88.9 0)
       (effects (font (size 1.27 1.27)) hide)
     )
@@
       (effects (font (size 1.27 1.27)) hide)
     )
-    (pin "2")
-    (pin "1")
+    (pin "1")
+    (pin "2")
     (instances
       (project "ez-bno055"
@@
       (effects (font (size 1.27 1.27)) hide)
     )
-    (pin "2")
-    (pin "1")
+    (pin "1")
+    (pin "2")
+    (pin "3")
     (pin "4")
-    (pin "3")
     (pin "5")
     (pin "6")
@@
     )
     (pin "1")
+    (pin "2")
+    (pin "3")
     (pin "4")
+    (pin "S1")
     (pin "S2")
-    (pin "3")
-    (pin "2")
-    (pin "S1")
     (instances
       (project "ez-bno055"
@@
     )
     (pin "1")
+    (pin "2")
+    (pin "3")
     (pin "4")
+    (pin "S1")
     (pin "S2")
-    (pin "3")
-    (pin "2")
-    (pin "S1")
     (instances
       (project "ez-bno055"
@@
       (effects (font (size 1.27 1.27)) hide)
     )
-    (pin "2")
-    (pin "1")
+    (pin "1")
+    (pin "2")
     (instances
       (project "ez-bno055"
@@
       (effects (font (size 1.27 1.27)) hide)
     )
-    (pin "2")
-    (pin "1")
+    (pin "1")
+    (pin "2")
     (instances
       (project "ez-bno055"
@@
       (effects (font (size 1.27 1.27)) hide)
     )
-    (pin "2")
-    (pin "1")
+    (pin "1")
+    (pin "2")
     (instances
       (project "ez-bno055"
@@
       (effects (font (size 1.27 1.27)) hide)
     )
+    (pin "1")
+    (pin "10")
+    (pin "11")
+    (pin "12")
+    (pin "13")
+    (pin "14")
+    (pin "15")
     (pin "16")
+    (pin "17")
+    (pin "18")
+    (pin "19")
+    (pin "2")
+    (pin "20")
+    (pin "21")
+    (pin "22")
+    (pin "23")
+    (pin "24")
+    (pin "25")
+    (pin "26")
+    (pin "27")
+    (pin "28")
+    (pin "3")
     (pin "4")
-    (pin "28")
-    (pin "18")
-    (pin "2")
-    (pin "19")
+    (pin "5")
     (pin "6")
-    (pin "25")
     (pin "7")
-    (pin "5")
-    (pin "27")
     (pin "8")
-    (pin "23")
-    (pin "14")
     (pin "9")
-    (pin "26")
-    (pin "15")
-    (pin "17")
-    (pin "22")
-    (pin "13")
-    (pin "11")
-    (pin "21")
-    (pin "3")
-    (pin "1")
-    (pin "24")
-    (pin "12")
-    (pin "10")
-    (pin "20")
     (instances
       (project "ez-bno055"
@@
       (effects (font (size 1.27 1.27)) hide)
     )
-    (pin "2")
-    (pin "1")
+    (pin "1")
+    (pin "2")
     (instances
       (project "ez-bno055"
@@
       (effects (font (size 1.27 1.27)) hide)
     )
-    (pin "2")
-    (pin "1")
+    (pin "1")
+    (pin "2")
     (instances
       (project "ez-bno055"
@@
     )
     (pin "1")
+    (pin "2")
+    (pin "3")
     (pin "4")
     (pin "5")
-    (pin "2")
-    (pin "3")
     (instances
       (project "ez-bno055"
@@
       (effects (font (size 1.27 1.27)) hide)
     )
-    (pin "2")
-    (pin "1")
+    (pin "1")
+    (pin "2")
     (instances
       (project "ez-bno055"
@@
       (effects (font (size 1.27 1.27)) hide)
     )
-    (pin "2")
-    (pin "1")
+    (pin "1")
+    (pin "2")
+    (pin "3")
     (pin "4")
-    (pin "3")
     (pin "5")
     (pin "6")
@@
       (effects (font (size 1.27 1.27)) hide)
     )
-    (pin "2")
-    (pin "1")
-    (instances
-      (project "ez-bno055"
+    (pin "1")
+    (pin "2")
+    (instances
+      (project "ez-bno055"
